File: Project Architecture.kicad_sch (KiCad schematic)
At the start: 0 parts

Commit message: First draft of schematic
Other:
- sheet Section A - Title A renamed MCU
- sheet Section B - Title B renamed IMU
- added sheet Connectors (Connectors.kicad_sch)
- added sheet Holes, Fiducials (Holes, Fiducials.kicad_sch)
- sheet IMU: file Section B - TItle B.kicad_sch -> IMU.kicad_sch
- sheet IMU ports: added {I2C2}; removed none
- sheet MCU: file Section A - Title A.kicad_sch -> MCU.kicad_sch
- sheet MCU ports: added {I2C2}, {SWD}; removed none
- note added: "Page 6"
- note added: "Page 7"
